Commit message: complete system v0.0

File: catkin_ws/src/bot_pkg/urdf/bot.urdf (robot description, URDF)
Before this commit: robot multipleshapes, 3 links, 2 joints
Links:
- link base_link: geometry visual box size=0.175 0.24 .02
- link l_wheel: geometry visual cylinder length=0.045 radius=0.05
- link r_wheel: geometry visual cylinder length=0.045 radius=0.05
Joints:
- joint base_to_l_wheel: origin xyz=-0.05 0 0.01 rpy=0 1.57075 0 -> xyz=-0.13 -0.03 0.00 rpy=0 1.57075 0; type static -> fixed
- joint base_to_r_wheel: origin xyz=0.05 0 0.01 rpy=0 -1.57075 0 -> xyz= 0.13 -0.03 0.00 rpy=0 -1.57075 0; type static -> fixed

File: catkin_ws/src/temp_urdf/sparkv_copy.urdf (robot description, URDF)
Before this commit: robot multipleshapes, 3 links, 2 joints
Joints:
- joint base_to_l_wheel: type static -> continuous
- joint base_to_r_wheel: type static -> continuous
